File: waker/main.sch (EAGLE design)
At the start: 46 parts, among them IC1 C8051F381-GM, IC3 N25Q512A, IC4 KC2016K, IC6 MPU-9250, P0.0 PTR1TP10R, SW2 PTR1TP10R, U1 MCP73831, U2 TPS61200

Commit message: Added MCU, Gyro and Flash memory
Parts:
- removed C12: 0.1u, reg,cap:C-1005
- removed IC4: KC2016K, Oscillator:KC2016K
- added FET1: DMN3404L, MOSFET:DMN3404L
- added MN, MP: PTR1TP10R, testpad:PTR1TP10R
- added R13, R14: 10k, reg,cap:R-1005
- added R15: 100k, reg,cap:R-1005
- added S1: (no value), SparkFun-Switches:MOMENTARY-SWITCH-SPST-2-SMD-4.6X2.8MM
- R1: device SparkFun-Resistors:RESISTORPTH-1/4W-VERT-KIT -> SparkFun-Resistors:2.0KOHM1/10W5%(0603)
Connections:
- removed net N$11: IC1G$1.P0.3/XTAL2, IC4.OUT
- new net N$10: FET1.D, MN.TP
- new net N$5: D2.A, IC1G$1.P0.1, R13.P$2, S1.3, S1.4
- new net N$6: D2.C, D4.C, R14.P$2, U2.EN
- new net N$7: D4.A, IC1G$1.P0.0
- new net N$8: FET1.G, IC1G$1.P0.2/XTAL1, R15.P$2
- net DGND: now also FET1.S, R13.P$1, R14.P$1, R15.P$1; no longer C12.P$1, IC4.GND
- net GND: now also R1.2; no longer R1.1
- net PROG: now also R1.1; no longer R1.2
- net VBAT: now also S1.1, S1.2; no longer U2.EN
- net VCC: now also MP.TP; no longer C12.P$2, IC4.EN, IC4.VCC
Other:
- moved on the sheet: D2, D4, R1

Commit message: Modified circuit
Parts:
- added R16: 10k, reg,cap:R-1005
- added R17: 100, reg,cap:R-1005
- R15: value 100k -> 10k
Connections:
- new net N$11: D2.A, R13.P$2, R16.P$2, S1.3, S1.4
- new net N$12: IC1G$1.P0.2/XTAL1
- new net PWM: IC1G$1.P2.6, R15.P$2, R17.P$2
- net N$5: now also R16.P$1; no longer D2.A, R13.P$2, S1.3, S1.4
- net N$8: now also R17.P$1; no longer IC1G$1.P0.2/XTAL1, R15.P$2
Other:
- moved on the sheet: FET1, MN, MP, R15
Changed lines of the file:
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@@
 <part name="GND4" library="supply2" library_urn="urn:adsk.eagle:library:372" deviceset="DGND" device=""/>
 <part name="FET1" library="MOSFET" deviceset="DMN3404L" device=""/>
-<part name="R15" library="reg,cap" deviceset="R-" device="1005" value="100k"/>
+<part name="R15" library="reg,cap" deviceset="R-" device="1005" value="10k"/>
 <part name="SUPPLY3" library="supply2" deviceset="DGND" device=""/>
 <part name="SUPPLY5" library="supply2" deviceset="DGND" device=""/>
@@
 <part name="MP" library="testpad" deviceset="PTR1" device="TP10R"/>
 <part name="+3V3" library="supply1" library_urn="urn:adsk.eagle:library:371" deviceset="VCC" device=""/>
+<part name="R16" library="reg,cap" deviceset="R-" device="1005" value="10k"/>
+<part name="R17" library="reg,cap" deviceset="R-" device="1005" value="100"/>
 </parts>
 <sheets>
@@
 <instance part="R14" gate="G$1" x="180.34" y="76.2" rot="R90"/>
 <instance part="GND4" gate="G$1" x="180.34" y="71.12"/>
-<instance part="FET1" gate="G$1" x="353.06" y="86.36" rot="MR0"/>
-<instance part="R15" gate="G$1" x="363.22" y="78.74" rot="R90"/>
-<instance part="SUPPLY3" gate="G$1" x="363.22" y="73.66"/>
-<instance part="SUPPLY5" gate="G$1" x="353.06" y="73.66"/>
+<instance part="FET1" gate="G$1" x="353.06" y="-73.66" rot="MR0"/>
+<instance part="R15" gate="G$1" x="375.92" y="-81.28" rot="R90"/>
+<instance part="SUPPLY3" gate="G$1" x="375.92" y="-86.36"/>
+<instance part="SUPPLY5" gate="G$1" x="353.06" y="-86.36"/>
 <instance part="R1" gate="G$1" x="76.2" y="0" rot="R270"/>
-<instance part="MN" gate="G$1" x="350.52" y="96.52" rot="R270"/>
-<instance part="MP" gate="G$1" x="350.52" y="104.14" rot="R270"/>
-<instance part="+3V3" gate="VCC" x="353.06" y="111.76"/>
+<instance part="MN" gate="G$1" x="350.52" y="-63.5" rot="R270"/>
+<instance part="MP" gate="G$1" x="350.52" y="-55.88" rot="R270"/>
+<instance part="+3V3" gate="VCC" x="353.06" y="-48.26"/>
+<instance part="R16" gate="G$1" x="193.04" y="86.36" rot="R180"/>
+<instance part="R17" gate="G$1" x="365.76" y="-76.2"/>
 </instances>
 <busses>
@@
 <pinref part="FET1" gate="G$1" pin="S"/>
 <pinref part="SUPPLY5" gate="G$1" pin="DGND"/>
-<wire x1="353.06" y1="81.28" x2="353.06" y2="76.2" width="0.1524" layer="91"/>
+<wire x1="353.06" y1="-78.74" x2="353.06" y2="-83.82" width="0.1524" layer="91"/>
 </segment>
 </net>
@@
 <segment>
 <pinref part="MP" gate="G$1" pin="TP"/>
-<wire x1="353.06" y1="104.14" x2="353.06" y2="109.22" width="0.1524" layer="91"/>
+<wire x1="353.06" y1="-55.88" x2="353.06" y2="-50.8" width="0.1524" layer="91"/>
 <pinref part="+3V3" gate="VCC" pin="VCC"/>
 </segment>
@@
 <net name="N$5" class="0">
 <segment>
-<pinref part="S1" gate="G$1" pin="3"/>
-<pinref part="S1" gate="G$1" pin="4"/>
-<wire x1="157.48" y1="83.82" x2="157.48" y2="81.28" width="0.1524" layer="91"/>
-<pinref part="R13" gate="G$1" pin="P$2"/>
-<wire x1="160.02" y1="81.28" x2="157.48" y2="81.28" width="0.1524" layer="91"/>
-<junction x="157.48" y="81.28"/>
-<pinref part="D2" gate="G$1" pin="A"/>
-<wire x1="160.02" y1="81.28" x2="167.64" y2="81.28" width="0.1524" layer="91"/>
-<junction x="160.02" y="81.28"/>
 <pinref part="IC1" gate="G$1" pin="P0.1"/>
 <wire x1="373.38" y1="66.04" x2="213.36" y2="66.04" width="0.1524" layer="91"/>
 <wire x1="213.36" y1="66.04" x2="213.36" y2="86.36" width="0.1524" layer="91"/>
-<wire x1="213.36" y1="86.36" x2="160.02" y2="86.36" width="0.1524" layer="91"/>
-<wire x1="160.02" y1="86.36" x2="160.02" y2="81.28" width="0.1524" layer="91"/>
+<wire x1="213.36" y1="86.36" x2="195.58" y2="86.36" width="0.1524" layer="91"/>
+<pinref part="R16" gate="G$1" pin="P$1"/>
 </segment>
 </net>
@@
 </segment>
 </net>
-<net name="N$8" class="0">
-<segment>
-<pinref part="FET1" gate="G$1" pin="G"/>
+<net name="PWM" class="0">
+<segment>
 <pinref part="R15" gate="G$1" pin="P$2"/>
-<wire x1="358.14" y1="83.82" x2="363.22" y2="83.82" width="0.1524" layer="91"/>
+<pinref part="IC1" gate="G$1" pin="P2.6"/>
+<wire x1="370.84" y1="-76.2" x2="375.92" y2="-76.2" width="0.1524" layer="91"/>
+<wire x1="396.24" y1="33.02" x2="396.24" y2="-76.2" width="0.1524" layer="91"/>
+<wire x1="396.24" y1="-76.2" x2="375.92" y2="-76.2" width="0.1524" layer="91"/>
+<junction x="375.92" y="-76.2"/>
+<label x="383.54" y="-76.2" size="1.778" layer="95"/>
+<pinref part="R17" gate="G$1" pin="P$2"/>
+</segment>
+</net>
+<net name="N$10" class="0">
+<segment>
+<pinref part="MN" gate="G$1" pin="TP"/>
+<pinref part="FET1" gate="G$1" pin="D"/>
+<wire x1="353.06" y1="-63.5" x2="353.06" y2="-68.58" width="0.1524" layer="91"/>
+</segment>
+</net>
+<net name="N$11" class="0">
+<segment>
+<pinref part="D2" gate="G$1" pin="A"/>
+<pinref part="S1" gate="G$1" pin="4"/>
+<pinref part="S1" gate="G$1" pin="3"/>
+<wire x1="157.48" y1="83.82" x2="157.48" y2="81.28" width="0.1524" layer="91"/>
+<junction x="157.48" y="81.28"/>
+<pinref part="R13" gate="G$1" pin="P$2"/>
+<wire x1="160.02" y1="81.28" x2="157.48" y2="81.28" width="0.1524" layer="91"/>
+<wire x1="160.02" y1="81.28" x2="167.64" y2="81.28" width="0.1524" layer="91"/>
+<junction x="160.02" y="81.28"/>
+<wire x1="160.02" y1="86.36" x2="160.02" y2="81.28" width="0.1524" layer="91"/>
+<wire x1="187.96" y1="86.36" x2="160.02" y2="86.36" width="0.1524" layer="91"/>
+<pinref part="R16" gate="G$1" pin="P$2"/>
+</segment>
+</net>
+<net name="N$12" class="0">
+<segment>
 <pinref part="IC1" gate="G$1" pin="P0.2/XTAL1"/>
 <wire x1="388.62" y1="81.28" x2="388.62" y2="83.82" width="0.1524" layer="91"/>
-<wire x1="388.62" y1="83.82" x2="363.22" y2="83.82" width="0.1524" layer="91"/>
-<junction x="363.22" y="83.82"/>
-</segment>
-</net>
-<net name="N$10" class="0">
-<segment>
-<pinref part="MN" gate="G$1" pin="TP"/>
-<pinref part="FET1" gate="G$1" pin="D"/>
-<wire x1="353.06" y1="96.52" x2="353.06" y2="91.44" width="0.1524" layer="91"/>
-</segment>
-</net>
+</segment>
+</net>
+<net name="N$8" class="0">
+<segment>
+<pinref part="R17" gate="G$1" pin="P$1"/>
+<pinref part="FET1" gate="G$1" pin="G"/>
+<wire x1="358.14" y1="-76.2" x2="363.22" y2="-76.2" width="0.1524" layer="91"/>
+</segment>
+</net>

Commit message: Puttin parts
Parts:
- removed C2CK, C2D, DGND, GND, P0.0: PTR1TP10R, testpad:PTR1TP10R
- removed C6: 10uF, CH_passive:CAP1206
- removed R6: 1.2M, SparkFun:RESISTOR0603-RES
- removed R7: 220k, SparkFun:RESISTOR0603-RES
- removed R8: 2M, SparkFun:RESISTOR0603-RES
- removed SJ1: (no value), SparkFun:SOLDERJUMPER_2WAYPASTE2&3
- added C12: 10uF, CH_passive:CAP1206
- added JP2: (no value), pinhead:PINHD-1X1
- added JP3: (no value), pinhead:PINHD-1X3
- added R18: (no value), rcl:R-US_R0402
- C2, C5: device SparkFun:CAP0603-CAP -> rcl:C-USC0402K
- R1, R4: device SparkFun-Resistors:2.0KOHM1/10W5%(0603) -> rcl:R-US_R0402
- R2, R5: device SparkFun:RESISTOR0603-RES -> rcl:R-US_R0402
- R3: device SparkFun-Resistors:330OHM1/10W1%(0603) -> rcl:R-US_R0402
- U2: value TPS61200 -> TPS61201
Connections:
- removed net 3.3V: R6.1, SJ1.1
- removed net 5V: R8.1, SJ1.3
- removed net FB: R7.2, SJ1.2, U2.FB
- net C2CK: now also JP3.3; no longer C2CK.TP
- net C2D: now also JP3.2; no longer C2D.TP
- net DGND: now also JP3.1; no longer DGND.TP, GND.TP
- net GND: now also C12.2; no longer C6.2, R7.1
- net N$15: now also JP2.1; no longer P0.0.TP
- net VBAT: now also C12.1; no longer C6.1
- net VCC: now also U2.FB; no longer R6.2, R8.2
Other:
- moved on the sheet: C1, C2, C5

Commit message: Modified parts places
Parts:
- removed R18: (no value), rcl:R-US_R0402
- removed SW2: PTR1TP10R, testpad:PTR1TP10R
Connections:
- removed net N$12: IC1G$1.P0.2/XTAL1
- removed net N$4: IC1G$1.P1.1, SW2.TP
Changed lines of the file:
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@@
 <part name="SUPPLY4" library="supply2" deviceset="DGND" device=""/>
 <part name="+3V1" library="supply1" library_urn="urn:adsk.eagle:library:371" deviceset="VCC" device=""/>
-<part name="SW2" library="testpad" deviceset="PTR1" device="TP10R"/>
 <part name="R11" library="reg,cap" deviceset="R-" device="1005" value="1k"/>
 <part name="+3V2" library="supply1" library_urn="urn:adsk.eagle:library:371" deviceset="VCC" device=""/>
@@
 <part name="JP2" library="pinhead" library_urn="urn:adsk.eagle:library:325" deviceset="PINHD-1X1" device="" package3d_urn="urn:adsk.eagle:package:22485/2"/>
 <part name="JP3" library="pinhead" library_urn="urn:adsk.eagle:library:325" deviceset="PINHD-1X3" device="" package3d_urn="urn:adsk.eagle:package:22458/2"/>
-<part name="R18" library="rcl" library_urn="urn:adsk.eagle:library:334" deviceset="R-US_" device="R0402" package3d_urn="urn:adsk.eagle:package:23547/2"/>
 <part name="C12" library="CH_passive" deviceset="CAP" device="1206" value="10uF"/>
 </parts>
@@
 <instance part="SUPPLY4" gate="G$1" x="292.1" y="33.02"/>
 <instance part="+3V1" gate="VCC" x="358.14" y="45.72"/>
-<instance part="SW2" gate="G$1" x="408.94" y="99.06" rot="R90"/>
 <instance part="R11" gate="G$1" x="337.82" y="33.02" rot="R90"/>
 <instance part="+3V2" gate="VCC" x="337.82" y="40.64"/>
@@
 <instance part="JP2" gate="G$1" x="375.92" y="0" rot="R90"/>
 <instance part="JP3" gate="A" x="312.42" y="10.16" rot="R180"/>
-<instance part="R18" gate="G$1" x="83.82" y="-22.86"/>
 <instance part="C12" gate="G$1" x="116.84" y="7.62" smashed="yes">
 <attribute name="NAME" x="119.38" y="10.16" size="1.778" layer="95"/>
@@
 </segment>
 </net>
-<net name="N$4" class="0">
-<segment>
-<wire x1="406.4" y1="81.28" x2="406.4" y2="99.06" width="0.1524" layer="91"/>
-<pinref part="IC1" gate="G$1" pin="P1.1"/>
-<pinref part="SW2" gate="G$1" pin="TP"/>
-</segment>
-</net>
 <net name="VCC" class="0">
 <segment>
@@
 </segment>
 </net>
-<net name="N$12" class="0">
-<segment>
-<pinref part="IC1" gate="G$1" pin="P0.2/XTAL1"/>
-<wire x1="388.62" y1="81.28" x2="388.62" y2="83.82" width="0.1524" layer="91"/>
-</segment>
-</net>
